File: led_lamp_pcb/led_lamp_pcb.kicad_sch (KiCad schematic)
At the start: 47 parts, among them J1 Conn_01x02_Male, J2 Conn_01x04_Male, J3 Screw_Terminal_01x02, J4 Screw_Terminal_01x02, J5 Screw_Terminal_01x02, J6 Screw_Terminal_01x02, K1 SANYOU_SRD_Form_C, Q1 NTR1P02, Q2 Si2302DS, SW1 SW_SPST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

Commit message: rev 1 as send to manufacturer
Parts:
- removed C2: 100n, symbol Device:C
- removed C5: 100m, symbol Device:C_Polarized
- removed D1: 5.6V, symbol Device:D_Zener
- removed Q1: NTR1P02, symbol Device:Q_PMOS_GSD
- removed R10, R3: 50k, symbol Device:R
- removed R11: 1k, symbol Device:R
- removed R4: 10k, symbol Device:R
- removed RV2: 10k, symbol Device:R_Potentiometer_Trim
- removed U1: LM393, symbol Comparator:LM393
- added C2: 0.47, proj_footprints:CHP5R5L504R-TW, symbol Device:C_Polarized
- added C3: 10u, Capacitor_SMD:C_0805_2012Metric_Pad1.18x1.45mm_HandSolder, symbol Device:C
- added D1, D3: 1N5817, Diode_SMD:D_SMA_Handsoldering, symbol Diode:1N5819
- added U1: TL331, Package_TO_SOT_SMD:SOT-23-5_HandSoldering, symbol Comparator:TL331
- C1, C6, C7: footprint (none) -> Capacitor_SMD:C_0805_2012Metric_Pad1.18x1.45mm_HandSolder
- C4: renamed from C3; footprint (none) -> Capacitor_SMD:C_0805_2012Metric_Pad1.18x1.45mm_HandSolder
- C5: renamed from C4; footprint (none) -> Capacitor_SMD:C_0805_2012Metric_Pad1.18x1.45mm_HandSolder
- D2: value 1N5819 -> 1N5817; footprint Diode_THT:D_DO-41_SOD81_P10.16mm_Horizontal -> Diode_SMD:D_SMA_Handsoldering
- J1: footprint (none) -> Connector_PinHeader_2.54mm:PinHeader_1x02_P2.54mm_Vertical
- J2: footprint (none) -> Connector_PinHeader_2.54mm:PinHeader_1x04_P2.54mm_Vertical
- J3, J4, J5, J6: footprint (none) -> TerminalBlock:TerminalBlock_bornier-2_P5.08mm
- Q1: renamed from Q2; footprint Package_TO_SOT_SMD:SOT-23 -> Package_TO_SOT_SMD:SOT-23_Handsoldering; Spice_Netlist_Enabled Y -> N
- R1: value 50k -> 100k; footprint (none) -> Resistor_SMD:R_0805_2012Metric_Pad1.20x1.40mm_HandSolder
- R10: renamed from R14; footprint (none) -> Resistor_SMD:R_0805_2012Metric_Pad1.20x1.40mm_HandSolder
- R11: renamed from R15; footprint (none) -> Resistor_SMD:R_0805_2012Metric_Pad1.20x1.40mm_HandSolder
- R12: renamed from R16; footprint (none) -> Resistor_SMD:R_0805_2012Metric_Pad1.20x1.40mm_HandSolder
- R13: renamed from R17; footprint (none) -> Resistor_SMD:R_0805_2012Metric_Pad1.20x1.40mm_HandSolder
- R14: renamed from R18; footprint (none) -> Resistor_SMD:R_0805_2012Metric_Pad1.20x1.40mm_HandSolder
- R15: renamed from R19; footprint (none) -> Resistor_SMD:R_0805_2012Metric_Pad1.20x1.40mm_HandSolder
- R2: value 10k -> 20k; footprint (none) -> Resistor_SMD:R_0805_2012Metric_Pad1.20x1.40mm_HandSolder
- R3: renamed from R8; value 10k -> 20k; footprint (none) -> Resistor_SMD:R_0805_2012Metric_Pad1.20x1.40mm_HandSolder
- R4: renamed from R9; footprint (none) -> Resistor_SMD:R_0805_2012Metric_Pad1.20x1.40mm_HandSolder
- R5, R6: footprint (none) -> Resistor_SMD:R_0805_2012Metric_Pad1.20x1.40mm_HandSolder
- R7: value 10k -> 10; footprint (none) -> Resistor_THT:R_Axial_DIN0207_L6.3mm_D2.5mm_P7.62mm_Horizontal
- R8: renamed from R12; footprint (none) -> Resistor_SMD:R_0805_2012Metric_Pad1.20x1.40mm_HandSolder
- R9: renamed from R13; footprint (none) -> Resistor_SMD:R_0805_2012Metric_Pad1.20x1.40mm_HandSolder
- RV1: footprint (none) -> Potentiometer_THT:Potentiometer_Piher_PT-10-V05_Vertical; Spice_Netlist_Enabled Y -> N
- SW1: footprint (none) -> Button_Switch_SMD:SW_Push_1P1T_NO_6x6mm_H9.5mm; Spice_Netlist_Enabled (none) -> N
- U3: footprint Package_TO_SOT_SMD:SOT-23-5 -> Package_TO_SOT_SMD:SOT-23-5_HandSoldering
- U4: footprint (none) -> Package_TO_SOT_SMD:SOT-23-5_HandSoldering; Spice_Netlist_Enabled (none) -> N
- V1, V3: Spice_Netlist_Enabled Y -> N; now left out of the parts list
- V2: now left out of the parts list
Connections:
- net +5V: now also D1.2 (A)
- net 3.3V: now also R3.2, U1.5 (V+); no longer R7.2
- net GND: now also C2.2, C3.2, U1.2 (V-)
- net P+5V: now also R7.2, D1.1 (K), D3.1 (K)
- net low_V: now also U1.4
- net at K1.2, Q1.3 (D): now also D3.2 (A); no longer D2.2 (A)
- net at R3.1, R4.2: now also U1.1 (-)
- net RX: now reaches U2.21 (GPIO3/RXD)
- net RX: now also J2.3 (Pin_3); no longer J2.2 (Pin_2)
- net TX: now reaches U2.22 (GPIO1/TXD)
- net TX: now also J2.2 (Pin_2); no longer J2.3 (Pin_3)
- net at R1.1, R2.2: now also U1.3 (+)
- net at R7.1: now also D2.2 (A), C2.1, C3.1; no longer R3.2
- no-connect marks 12 -> 11
Other:
- moved on the sheet: C4, C5, R1, R2, R3, R4, RV1, U3
